Commit message: controller manager initializes

File: install/rl12dof_urdf_description/share/rl12dof_urdf_description/urdf/rl12dof_ros2_control.xacro (robot description, xacro)
@@ -1,90 +1,93 @@
-<?xml version="1.0" encoding="utf-8"?>
-<robot name="quadruped" xmlns:xacro="http://www.ros.org/wiki/xacro">
-    <ros2_control name="quadruped_hardware/CANMotorDriver_HR" type="system" >
-        <hardware>
-            <plugin>quadruped_hardware/CANMotor</plugin>
-            <param name="joint_name">link1_to_base</param>
-            <param name="can_bus" >can0</param>
-            <param name="can_id" >1</param>
-            <param name="flip" >true</param>
-            <param name="effort_limit" >12.0</param>
-            <param name="command_type" >radian</param>
-            <param name="frequency" >50.0</param>
-            <param name="zero_position_offset" >0</param>
-            <param name="min_position_limit" >-3.13</param>
-            <param name="max_position_limit" >0.531</param>
-        </hardware>
-        <joint name="link1_to_base">
-            <command_interface name="position"/>
-            <command_interface name="velocity"/>
-            <command_interface name="effort"/>
-            <command_interface name="kp"/>
-            <command_interface name="kd"/>
-            <command_interface name="m_state"/>
-            <command_interface name="flip"/>
-            <state_interface   name="position"/>
-            <state_interface   name="velocity"/>
-            <state_interface   name="effort"/>
-            <state_interface   name="m_state"/>
-            <state_interface   name="flip"/>
-        </joint>
-    </ros2_control>
-    <ros2_control name="quadruped_hardware/CANMotorDriver_HP" type="system">
-        <hardware>
-            <plugin>quadruped_hardware/CANMotor</plugin>
-            <param name="joint_name">link2_to_link1</param>
-            <param name="can_bus" >can0</param>
-            <param name="can_id" >2</param>
-            <param name="flip" >true</param>
-            <param name="effort_limit" >12.0</param>
-            <param name="command_type" >radian</param>
-            <param name="frequency" >50.0</param>
-            <param name="zero_position_offset" >0</param>
-            <param name="min_position_limit" >-4.0</param>
-            <param name="max_position_limit" >0.2</param>
-        </hardware>
-        <joint name="link2_to_link1">
-            <command_interface name="position"/>
-            <command_interface name="velocity"/>
-            <command_interface name="effort"/>
-            <command_interface name="kp"/>
-            <command_interface name="kd"/>
-            <command_interface name="m_state"/>
-            <command_interface name="flip"/>
-            <state_interface   name="position"/>
-            <state_interface   name="velocity"/>
-            <state_interface   name="effort"/>
-            <state_interface   name="m_state"/>
-            <state_interface   name="flip"/>
-        </joint>
-    </ros2_control>
-    <ros2_control name="quadruped_hardware/CANMotorDriver_KP" type="system" >
-        <hardware>
-            <plugin>quadruped_hardware/CANMotor</plugin>
-            <param name="joint_name">link3_to_link2</param>
-            <param name="can_bus" >can0</param>
-            <param name="can_id" >3</param>
-            <param name="flip" >true</param>
-            <param name="effort_limit" >12.0</param>
-            <param name="command_type" >radian</param>
-            <param name="frequency" >50.0</param>
-            <param name="zero_position_offset" >0</param>
-            <param name="min_position_limit" >-0.531</param>
-            <param name="max_position_limit" >3.131</param>
-        </hardware>
-        <joint name="link3_to_link2">
-            <command_interface name="position"/>
-            <command_interface name="velocity"/>
-            <command_interface name="effort"/>
-            <command_interface name="kp"/>
-            <command_interface name="kd"/>
-            <command_interface name="m_state"/>
-            <command_interface name="flip"/>
-            <state_interface   name="position"/>
-            <state_interface   name="velocity"/>
-            <state_interface   name="effort"/>
-            <state_interface   name="m_state"/>
-            <state_interface   name="flip"/>
-        </joint>
-    </ros2_control>
+<?xml version="1.0"?>
+<robot xmlns:xacro="http://www.ros.org/wiki/xacro">
+  <!-- HIP MOTOR -->
+  <ros2_control name="hip_roll" type="system">
+    <hardware>
+      <plugin>quadruped_hardware/CANMotor</plugin>
+      <param name="joint_name">link1_to_base</param>
+      <param name="can_bus">can0</param>
+      <param name="can_id">18</param>
+      <param name="flip">true</param>
+      <param name="effort_limit">12.0</param>
+      <param name="command_type">radian</param>
+      <param name="frequency">50.0</param>
+      <param name="zero_position_offset">0</param>
+      <param name="min_position_limit">-1.57</param>
+      <param name="max_position_limit">1.57</param>
+    </hardware>
+    <joint name="link1_to_base">
+      <command_interface name="position"/>
+      <command_interface name="velocity"/>
+      <command_interface name="effort"/>
+      <command_interface name="kp"/>
+      <command_interface name="kd"/>
+      <command_interface name="m_state"/>
+      <command_interface name="flip"/>
+      <state_interface name="position"/>
+      <state_interface name="velocity"/>
+      <state_interface name="effort"/>
+      <state_interface name="m_state"/>
+      <state_interface name="flip"/>
+    </joint>
+  </ros2_control>
+  <!-- THIGH MOTOR -->
+  <ros2_control name="hip_pitch" type="system">
+    <hardware>
+      <plugin>quadruped_hardware/CANMotor</plugin>
+      <param name="joint_name">link2_to_link1</param>
+      <param name="can_bus">can0</param>
+      <param name="can_id">19</param>
+      <param name="flip">true</param>
+      <param name="effort_limit">12.0</param>
+      <param name="command_type">radian</param>
+      <param name="frequency">50.0</param>
+      <param name="zero_position_offset">0</param>
+      <param name="min_position_limit">0.0</param>
+      <param name="max_position_limit">6.28</param>
+    </hardware>
+    <joint name="link2_to_link1">
+      <command_interface name="position"/>
+      <command_interface name="velocity"/>
+      <command_interface name="effort"/>
+      <command_interface name="kp"/>
+      <command_interface name="kd"/>
+      <command_interface name="m_state"/>
+      <command_interface name="flip"/>
+      <state_interface name="position"/>
+      <state_interface name="velocity"/>
+      <state_interface name="effort"/>
+      <state_interface name="m_state"/>
+      <state_interface name="flip"/>
+    </joint>
+  </ros2_control>
+  <!-- KNEE MOTOR -->
+  <ros2_control name="knee_pitch" type="system">
+    <hardware>
+      <plugin>quadruped_hardware/CANMotor</plugin>
+      <param name="joint_name">link3_to_link2</param>
+      <param name="can_bus">can0</param>
+      <param name="can_id">20</param>
+      <param name="flip">true</param>
+      <param name="effort_limit">12.0</param>
+      <param name="command_type">radian</param>
+      <param name="frequency">50.0</param>
+      <param name="zero_position_offset">0</param>
+      <param name="min_position_limit">0.0</param>
+      <param name="max_position_limit">2.35</param>
+    </hardware>
+    <joint name="link3_to_link2">
+      <command_interface name="position"/>
+      <command_interface name="velocity"/>
+      <command_interface name="effort"/>
+      <command_interface name="kp"/>
+      <command_interface name="kd"/>
+      <command_interface name="m_state"/>
+      <command_interface name="flip"/>
+      <state_interface name="position"/>
+      <state_interface name="velocity"/>
+      <state_interface name="effort"/>
+      <state_interface name="m_state"/>
+      <state_interface name="flip"/>
+    </joint>
+  </ros2_control>
 </robot>

File: src/rl12dof_urdf_description/urdf/rl12dof_ros2_control.xacro (robot description, xacro)
@@ -1,90 +1,93 @@
-<?xml version="1.0" encoding="utf-8"?>
-<robot name="quadruped" xmlns:xacro="http://www.ros.org/wiki/xacro">
-    <ros2_control name="quadruped_hardware/CANMotorDriver_HR" type="system" >
-        <hardware>
-            <plugin>quadruped_hardware/CANMotor</plugin>
-            <param name="joint_name">link1_to_base</param>
-            <param name="can_bus" >can0</param>
-            <param name="can_id" >1</param>
-            <param name="flip" >true</param>
-            <param name="effort_limit" >12.0</param>
-            <param name="command_type" >radian</param>
-            <param name="frequency" >50.0</param>
-            <param name="zero_position_offset" >0</param>
-            <param name="min_position_limit" >-1.57</param>
-            <param name="max_position_limit" >1.57</param>
-        </hardware>
-        <joint name="link1_to_base">
-            <command_interface name="position"/>
-            <command_interface name="velocity"/>
-            <command_interface name="effort"/>
-            <command_interface name="kp"/>
-            <command_interface name="kd"/>
-            <command_interface name="m_state"/>
-            <command_interface name="flip"/>
-            <state_interface   name="position"/>
-            <state_interface   name="velocity"/>
-            <state_interface   name="effort"/>
-            <state_interface   name="m_state"/>
-            <state_interface   name="flip"/>
-        </joint>
-    </ros2_control>
-    <ros2_control name="quadruped_hardware/CANMotorDriver_HP" type="system">
-        <hardware>
-            <plugin>quadruped_hardware/CANMotor</plugin>
-            <param name="joint_name">link2_to_link1</param>
-            <param name="can_bus" >can0</param>
-            <param name="can_id" >2</param>
-            <param name="flip" >true</param>
-            <param name="effort_limit" >12.0</param>
-            <param name="command_type" >radian</param>
-            <param name="frequency" >50.0</param>
-            <param name="zero_position_offset" >0</param>
-            <param name="min_position_limit" >0.0</param>
-            <param name="max_position_limit" >6.28</param>
-        </hardware>
-        <joint name="link2_to_link1">
-            <command_interface name="position"/>
-            <command_interface name="velocity"/>
-            <command_interface name="effort"/>
-            <command_interface name="kp"/>
-            <command_interface name="kd"/>
-            <command_interface name="m_state"/>
-            <command_interface name="flip"/>
-            <state_interface   name="position"/>
-            <state_interface   name="velocity"/>
-            <state_interface   name="effort"/>
-            <state_interface   name="m_state"/>
-            <state_interface   name="flip"/>
-        </joint>
-    </ros2_control>
-    <ros2_control name="quadruped_hardware/CANMotorDriver_KP" type="system" >
-        <hardware>
-            <plugin>quadruped_hardware/CANMotor</plugin>
-            <param name="joint_name">link3_to_link2</param>
-            <param name="can_bus" >can0</param>
-            <param name="can_id" >3</param>
-            <param name="flip" >true</param>
-            <param name="effort_limit" >12.0</param>
-            <param name="command_type" >radian</param>
-            <param name="frequency" >50.0</param>
-            <param name="zero_position_offset" >0</param>
-            <param name="min_position_limit" >0.0</param>
-            <param name="max_position_limit" >2.35</param>
-        </hardware>
-        <joint name="link3_to_link2">
-            <command_interface name="position"/>
-            <command_interface name="velocity"/>
-            <command_interface name="effort"/>
-            <command_interface name="kp"/>
-            <command_interface name="kd"/>
-            <command_interface name="m_state"/>
-            <command_interface name="flip"/>
-            <state_interface   name="position"/>
-            <state_interface   name="velocity"/>
-            <state_interface   name="effort"/>
-            <state_interface   name="m_state"/>
-            <state_interface   name="flip"/>
-        </joint>
-    </ros2_control>
+<?xml version="1.0"?>
+<robot xmlns:xacro="http://www.ros.org/wiki/xacro">
+  <!-- HIP MOTOR -->
+  <ros2_control name="hip_roll" type="system">
+    <hardware>
+      <plugin>quadruped_hardware/CANMotor</plugin>
+      <param name="joint_name">link1_to_base</param>
+      <param name="can_bus">can0</param>
+      <param name="can_id">18</param>
+      <param name="flip">true</param>
+      <param name="effort_limit">12.0</param>
+      <param name="command_type">radian</param>
+      <param name="frequency">50.0</param>
+      <param name="zero_position_offset">0</param>
+      <param name="min_position_limit">-1.57</param>
+      <param name="max_position_limit">1.57</param>
+    </hardware>
+    <joint name="link1_to_base">
+      <command_interface name="position"/>
+      <command_interface name="velocity"/>
+      <command_interface name="effort"/>
+      <command_interface name="kp"/>
+      <command_interface name="kd"/>
+      <command_interface name="m_state"/>
+      <command_interface name="flip"/>
+      <state_interface name="position"/>
+      <state_interface name="velocity"/>
+      <state_interface name="effort"/>
+      <state_interface name="m_state"/>
+      <state_interface name="flip"/>
+    </joint>
+  </ros2_control>
+  <!-- THIGH MOTOR -->
+  <ros2_control name="hip_pitch" type="system">
+    <hardware>
+      <plugin>quadruped_hardware/CANMotor</plugin>
+      <param name="joint_name">link2_to_link1</param>
+      <param name="can_bus">can0</param>
+      <param name="can_id">19</param>
+      <param name="flip">true</param>
+      <param name="effort_limit">12.0</param>
+      <param name="command_type">radian</param>
+      <param name="frequency">50.0</param>
+      <param name="zero_position_offset">0</param>
+      <param name="min_position_limit">0.0</param>
+      <param name="max_position_limit">6.28</param>
+    </hardware>
+    <joint name="link2_to_link1">
+      <command_interface name="position"/>
+      <command_interface name="velocity"/>
+      <command_interface name="effort"/>
+      <command_interface name="kp"/>
+      <command_interface name="kd"/>
+      <command_interface name="m_state"/>
+      <command_interface name="flip"/>
+      <state_interface name="position"/>
+      <state_interface name="velocity"/>
+      <state_interface name="effort"/>
+      <state_interface name="m_state"/>
+      <state_interface name="flip"/>
+    </joint>
+  </ros2_control>
+  <!-- KNEE MOTOR -->
+  <ros2_control name="knee_pitch" type="system">
+    <hardware>
+      <plugin>quadruped_hardware/CANMotor</plugin>
+      <param name="joint_name">link3_to_link2</param>
+      <param name="can_bus">can0</param>
+      <param name="can_id">20</param>
+      <param name="flip">true</param>
+      <param name="effort_limit">12.0</param>
+      <param name="command_type">radian</param>
+      <param name="frequency">50.0</param>
+      <param name="zero_position_offset">0</param>
+      <param name="min_position_limit">0.0</param>
+      <param name="max_position_limit">2.35</param>
+    </hardware>
+    <joint name="link3_to_link2">
+      <command_interface name="position"/>
+      <command_interface name="velocity"/>
+      <command_interface name="effort"/>
+      <command_interface name="kp"/>
+      <command_interface name="kd"/>
+      <command_interface name="m_state"/>
+      <command_interface name="flip"/>
+      <state_interface name="position"/>
+      <state_interface name="velocity"/>
+      <state_interface name="effort"/>
+      <state_interface name="m_state"/>
+      <state_interface name="flip"/>
+    </joint>
+  </ros2_control>
 </robot>
